File: Hardware/Galia.kicad_pcb (KiCad board)
At the start: 2 copper layers, 285.2 x 133.6 mm, 140 parts, among them J1 Bat, J2 OLED, J3 Interconnect, J4 Bat, J5 Trackball, J6 OLED, J7 Interconnect_R, SW1 MX, SW10 MX, SW11 MX, SW12 MX, SW13 MX, SW14 MX, SW15 MX, SW16 MX, SW17 MX, SW18 MX, SW19 MX, SW2 MX, SW20 MX, SW21 MX, SW22 MX, SW23 MX, SW24 MX, SW25 MX, SW26 MX, SW27 MX, SW28 MX, SW29 MX, SW3 MX, SW30 MX, SW31 MX, SW32 MX, SW33 MX, SW34 Encoder, SW35 Reset, SW36 MX, SW37 MX, SW38 MX, SW39 MX, SW4 MX, SW40 MX, SW41 MX, SW42 MX, SW43 MX, SW44 MX, SW45 MX, SW46 MX, SW47 MX, SW48 MX, SW49 MX, SW5 MX, SW50 MX, SW51 MX, SW52 MX, SW53 MX, SW54 MX, SW55 MX, SW56 MX, SW57 MX, SW58 MX, SW59 MX, SW6 MX, SW60 MX, SW61 MX, SW62 MX, SW63 MX, SW64 Reset, SW7 MX, SW8 MX, SW9 MX, U1 ProMicro, U2 ProMicro

Commit message: Updated silkscreen
Parts:
- added G1: Art, Cantaloupe:Catmelon, B.Cu at (258.8, 119.0)
- added G2: Art, Cantaloupe:Catmelon, B.Cu at (129.4, 119.0)
- added REF**: MountingHole_2.2mm_M2_Pad, MountingHole:MountingHole_2.2mm_M2_Pad, F.Cu at (56.4, 103.2)
- added REF**: MountingHole_2.2mm_M2_Pad, MountingHole:MountingHole_2.2mm_M2_Pad, F.Cu at (174.6, 117.5)
- added REF**: MountingHole_2.2mm_M2_Pad, MountingHole:MountingHole_2.2mm_M2_Pad, F.Cu at (174.6, 60.3)
- added REF**: Breakaway_Tabs, Custom Parts:Breakaway_Tabs, F.Cu at (195.3, 127.0)
- added REF**: Breakaway_Tabs, Custom Parts:Breakaway_Tabs, F.Cu at (193.7, 127.0)
- added REF**: Breakaway_Tabs, Custom Parts:Breakaway_Tabs, F.Cu at (195.3, 108.0)
- added REF**: Breakaway_Tabs, Custom Parts:Breakaway_Tabs, F.Cu at (193.7, 108.0)
- added REF**: Breakaway_Tabs, Custom Parts:Breakaway_Tabs, F.Cu at (195.3, 88.9)
- added REF**: Breakaway_Tabs, Custom Parts:Breakaway_Tabs, F.Cu at (193.7, 88.9)
- added REF**: Breakaway_Tabs, Custom Parts:Breakaway_Tabs, F.Cu at (195.3, 69.8)
- added REF**: Breakaway_Tabs, Custom Parts:Breakaway_Tabs, F.Cu at (193.7, 69.8)
- added REF**: MountingHole_2.2mm_M2_Pad, MountingHole:MountingHole_2.2mm_M2_Pad, F.Cu at (332.6, 103.2)
- added REF**: Breakaway_Tabs, Custom Parts:Breakaway_Tabs, F.Cu at (195.3, 50.8)
- added REF**: Breakaway_Tabs, Custom Parts:Breakaway_Tabs, F.Cu at (193.7, 50.8)
- added REF**: MountingHole_2.2mm_M2_Pad, MountingHole:MountingHole_2.2mm_M2_Pad, F.Cu at (302.4, 140.5)
- added REF**: MountingHole_2.2mm_M2_Pad, MountingHole:MountingHole_2.2mm_M2_Pad, F.Cu at (271.5, 112.7)
- added REF**: MountingHole_2.2mm_M2_Pad, MountingHole:MountingHole_2.2mm_M2_Pad, F.Cu at (290.5, 57.1)
- added REF**: MountingHole_2.2mm_M2_Pad, MountingHole:MountingHole_2.2mm_M2_Pad, F.Cu at (214.3, 117.5)
- added REF**: MountingHole_2.2mm_M2_Pad, MountingHole:MountingHole_2.2mm_M2_Pad, F.Cu at (214.3, 60.3)
- added REF**: MountingHole_2.2mm_M2_Pad, MountingHole:MountingHole_2.2mm_M2_Pad, F.Cu at (117.5, 112.7)
- added REF**: MountingHole_2.2mm_M2_Pad, MountingHole:MountingHole_2.2mm_M2_Pad, F.Cu at (98.4, 57.1)
- J1, J4, J5: moved to B.Cu
- moved J1 7.96 mm to (319.9, 106.4), turned to 270 degrees
- moved J4 7.94 mm to (70.6, 106.4), turned to 270 degrees
- moved D22 0.59 mm to (288.9, 46.0)
- moved D23 0.59 mm to (288.9, 65.1)
- moved D24 0.59 mm to (288.9, 84.1)
- moved D25 0.59 mm to (288.9, 103.2)
- moved D26 0.59 mm to (303.4, 130.9)
- moved D28 0.59 mm to (308.0, 49.2)
- moved D29 0.59 mm to (308.0, 68.3)
- moved D30 0.59 mm to (308.0, 87.3)
- moved D31 0.59 mm to (308.0, 106.4)
- moved D33 0.59 mm to (322.8, 140.7)
- moved J2 0.59 mm to (323.5, 72.0)
- moved R1 0.59 mm to (319.9, 81.0)
- moved REF** 0.59 mm to (315.5, 72.5)
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Routing:
- net Net-(J4-Pad2): track 69.5 -> 77.9 mm
- net Net-(J1-Pad2): track 70.4 -> 78.3 mm
- net GND1: track 154.5 -> 161.5 mm
- net COL1_R: track 280.4 -> 274.6 mm, vias 1 -> 0
- net COL4_R: track 238.9 -> 242.9 mm
- net GND3: track 167.4 -> 170.5 mm
- net SCLK: track 79.5 -> 77.0 mm
- net ROW1_R: track 153.3 -> 151.1 mm
- net COL5_R: track 179.1 -> 177.0 mm
- net ROW5_R: track 240.4 -> 238.5 mm
- net COL3_R: track 238.6 -> 237.1 mm, vias 1 -> 0
- net COL2: track 269.5 -> 268.1 mm
- net MISO: track 64.6 -> 65.7 mm
- net COL2_R: track 260.6 -> 260.0 mm, vias 1 -> 0
Other:
- board size 285.2 x 133.6 mm -> 285.7 x 133.6 mm
- board text added: "Galia Keyboard Left Hand Side V1.0 Designed By Aria"
- board text added: "Galia Keyboard Right Hand Side V1.0 Designed By Aria"
- board text added: "JLCJLCJLCJLC"
- board text added: "OLED"

Commit message: Added spot for TP4056 charger
Parts:
- J1, J4: value Bat -> TP4056; footprint Galia:Battery_Solder_Points -> Galia:TP4056-18650
- moved J4 10.7 mm to (64.6, 97.6), turned to 0 degrees
- moved J1 9.86 mm to (324.4, 97.6), turned to 180 degrees
- moved R1 6.83 mm to (314.3, 77.0)
- moved SW35 6.83 mm to (314.3, 83.3)
- moved REF** 6.35 mm to (56.4, 109.5)
- moved REF** 6.35 mm to (332.6, 109.5)
- moved R2 5.61 mm to (74.6, 77.1)
- moved SW64 5.61 mm to (74.6, 83.3)
- moved J3 4.01 mm to (338.3, 82.5)
- moved J7 4.01 mm to (50.6, 82.5)
- moved J6 0.32 mm to (65.4, 71.9)
Connections:
- J1 pad 1: GND1 -> Net-(J1-Pad1)
- J1 pad 2: Net-(J1-Pad2) -> GND1
- J4 pad 1: GND3 -> Net-(J4-Pad1)
- J4 pad 2: Net-(J4-Pad2) -> GND3
- U1 pad 24: Net-(J1-Pad2) -> RAW
- U2 pad 24: Net-(J4-Pad2) -> RAW_R
Routing:
- net Net-(J1-Pad2): track 78.3 -> 0.00 mm
- net Net-(J4-Pad2): track 77.9 -> 0.00 mm
- net RAW_R: track 0.00 -> 76.9 mm, vias 0 -> 2
- net RAW: track 0.00 -> 71.7 mm
- net GND1: track 161.5 -> 185.5 mm, vias 1 -> 0
- net VDD: track 105.7 -> 119.5 mm
- net CS: track 56.4 -> 69.1 mm
- net GND3: track 170.5 -> 182.5 mm, vias 3 -> 2
- net RESET: track 69.9 -> 61.5 mm, vias 2 -> 1
- net RESET_R: track 59.8 -> 52.3 mm
- net MOSI: track 61.0 -> 66.8 mm
- net DATA: track 62.1 -> 56.5 mm
- net VCC: track 68.5 -> 73.4 mm
- net DATA_R: track 53.5 -> 49.8 mm
- net ROW3_R: track 194.7 -> 197.8 mm
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Other:
- outline, holes or cut-outs redrawn

Commit message: Updated readme and added renders
Parts:
- J1, J4: moved to F.Cu
- moved R1 9.53 mm to (323.9, 77.0)
- moved SW35 9.53 mm to (323.9, 83.3)
- moved R2 9.52 mm to (65.1, 77.1)
- moved SW64 9.52 mm to (65.1, 83.3)
- moved U1 1.41 mm to (323.5, 50.5)
- moved U2 1.41 mm to (65.4, 50.3)
- moved REF** 0.32 mm to (73.4, 72.3)
- moved REF** 0.32 mm to (57.4, 72.3)
- moved J3 0.30 mm to (338.3, 82.2)
- moved J7 0.30 mm to (50.6, 82.2)
Routing:
- net RAW_R: track 76.9 -> 60.1 mm
- net RAW: track 71.7 -> 87.1 mm
- net VCC: track 73.4 -> 58.9 mm
- net GND3: track 182.5 -> 194.2 mm, vias 2 -> 4
- net RESET_R: track 52.3 -> 63.5 mm
- net GND1: track 185.5 -> 195.9 mm, vias 0 -> 1
- net ROW3_R: track 197.8 -> 204.8 mm
- net RESET: track 61.5 -> 55.5 mm
- net CS: track 69.1 -> 65.7 mm
- net VDD: track 119.5 -> 116.7 mm
- net MOSI: track 66.8 -> 63.9 mm
- net MISO: track 67.5 -> 64.7 mm
- net SCLK: track 76.8 -> 74.0 mm
- net SCL: track 29.9 -> 27.6 mm
- net DATA: track 56.5 -> 54.3 mm
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Other:
- outline, holes or cut-outs redrawn

Commit message: Changed reset switch footprint and position, removed pull-up resistor
Parts:
- removed R1, R2: 10k, Resistor_SMD:R_0603_1608Metric_Pad1.05x0.95mm_HandSolder
- SW35, SW64: footprint Button_Switch_SMD:SW_SPST_TL3342 -> Galia:Switch_Tactile_SPST_Angled_MJTP1117
- moved SW35 50.5 mm to (308.3, 35.3), turned to 180 degrees
- moved SW64 50.5 mm to (80.6, 35.3), turned to 180 degrees
Connections:
- SW35 pad 2: GND1 -> GND2
- U1 pad 3: Net-(U1-Pad3) -> GND2
Routing:
- net RESET_R: track 63.5 -> 12.7 mm, vias 1 -> 0
- net RESET: track 55.5 -> 92.6 mm, vias 1 -> 2
- net GND1: track 195.9 -> 161.4 mm
- net GND3: track 194.2 -> 219.3 mm, vias 4 -> 2
- net GND2: track 0.00 -> 16.2 mm, vias 0 -> 1
- net ROW3_R: track 204.8 -> 197.3 mm
- net VDD: track 116.7 -> 110.9 mm
- net VCC: track 58.9 -> 56.0 mm
- net RAW: track 87.1 -> 88.6 mm
- net ROW1_R: track 151.6 -> 152.5 mm
- net ROW5_R: track 241.8 -> 241.2 mm
- net ROW4_R: track 221.1 -> 220.5 mm
